Commit message: Update

File: tao_description/urdf/tao.urdf (robot description, URDF)
Before this commit: robot tao, 4 links, 3 joints
Links:
- removed link laser_link
- added link laser_frame, mass 0.073084; collision mesh filename=package://tao_description/meshes/laser_link.STL; visual mesh filename=package://tao_description/meshes/laser_link.STL
Joints:
- joint laser_joint: child laser_link -> laser_frame
- joint right_joint: origin xyz=0 -0.145 0.028 rpy=1.5708 1.2246E-16 -7.3956E-32 -> xyz=0 -0.145 0.028 rpy=1.5708 0 0
